File: kicad-pcb/krunchboard-v2/krunchboard-90.kicad_pcb (KiCad board)
At the start: 2 copper layers, 324 x 122.1 mm, 189 parts, among them J1 USB_C_Receptacle_USB2.0_16P, SW1 SW_Push_45deg, SW10 SW_Push_45deg, SW11 SW_Push_45deg, SW12 SW_Push_45deg, SW13 SW_Push_45deg, SW14 SW_Push_45deg, SW15 SW_Push_45deg, SW16 SW_Push_45deg, SW17 RotaryEncoder_Switch, SW18 SW_Push_45deg, SW19 SW_Push_45deg, SW2 SW_Push_45deg, SW20 SW_Push_45deg, SW21 SW_Push_45deg, SW22 SW_Push_45deg, SW23 SW_Push_45deg, SW24 SW_Push_45deg, SW25 SW_Push_45deg, SW26 SW_Push_45deg, SW27 SW_Push_45deg, SW28 SW_Push_45deg, SW29 SW_Push_45deg, SW3 SW_Push_45deg, SW30 SW_Push_45deg, SW31 SW_Push_45deg, SW32 SW_Push_45deg, SW33 SW_Push_45deg, SW34 SW_Push_45deg, SW35 SW_Push_45deg, SW36 SW_Push_45deg, SW37 SW_Push_45deg, SW38 SW_Push_45deg, SW39 SW_Push_45deg, SW4 SW_Push_45deg, SW40 SW_Push_45deg, SW41 SW_Push_45deg, SW42 SW_Push_45deg, SW43 SW_Push_45deg, SW44 SW_Push_45deg, SW45 SW_Push_45deg, SW46 SW_Push_45deg, SW47 SW_Push_45deg, SW48 SW_Push_45deg, SW49 SW_Push_45deg, SW5 SW_Push_45deg, SW50 SW_Push_45deg, SW51 SW_Push_45deg, SW52 SW_Push_45deg, SW53 SW_Push_45deg, SW54 SW_Push_45deg, SW55 SW_Push_45deg, SW56 SW_Push_45deg, SW57 SW_Push_45deg, SW58 SW_Push_45deg, SW59 SW_Push_45deg, SW6 SW_Push_45deg, SW60 SW_Push_45deg, SW61 SW_Push_45deg, SW62 SW_Push_45deg, SW63 SW_Push_45deg, SW64 SW_Push_45deg, SW65 SW_Push_45deg, SW66 SW_Push_45deg, SW67 SW_Push_45deg, SW68 SW_Push_45deg, SW69 SW_Push_45deg, SW7 SW_Push_45deg, SW70 SW_Push_45deg, SW71 SW_Push_45deg, SW72 SW_Push_45deg, SW73 SW_Push_45deg, SW74 SW_Push_45deg, SW75 SW_Push_45deg, SW76 SW_Push_45deg, SW77 SW_Push_45deg, SW78 SW_Push_45deg, SW79 SW_Push_45deg, SW8 SW_Push_45deg, SW80 SW_Push_45deg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

Commit message: updated pcb traces, firmware
Parts:
- moved A1 57.5 mm to (139.1, 185.6)
- moved D20 57.5 mm to (96.7, 115.5)
- moved D23 57.5 mm to (153.8, 115.5)
- moved D25 57.5 mm to (191.9, 115.5)
- moved D27 57.5 mm to (230.0, 115.5)
- moved D28 57.5 mm to (249.1, 115.5)
- moved D67 57.5 mm to (120.4, 170.5)
- moved D69 57.5 mm to (158.5, 170.5)
- moved D70 57.5 mm to (177.6, 172.7)
- moved D72 57.5 mm to (215.7, 172.7)
- moved D74 57.5 mm to (253.8, 172.7)
- moved D77 57.5 mm to (325.3, 172.7)
- moved R1 57.5 mm to (311.2, 81.9)
- moved SW53 57.5 mm to (124.6, 150.7)
- moved SW55 57.5 mm to (162.7, 150.7)
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Routing:
- net C12: track 249.6 -> 248.7 mm
- net Net-(A1-RUN): track 62.6 -> 61.7 mm
- net ENCB: track 283.8 -> 282.9 mm
- net C11: track 229.1 -> 228.2 mm
- net C10: track 207.5 -> 206.6 mm
- net C13: track 282.0 -> 281.1 mm
- net C1: track 157.9 -> 158.6 mm
- net C2: track 137.0 -> 137.5 mm
- net R4: track 319.5 -> 319.8 mm, vias 12 -> 10

Commit message: updated case,plate (added 4 extra mounting hole in center), updated pcb to prod v1
Parts:
- added G***: LOGO, LOGO, B.Cu at (207.3, 186.5)
- R1, R2: value R512 -> R512/R472; footprint Resistor_SMD:R_0402_1005Metric_Pad0.72x0.64mm_HandSolder -> Resistor_SMD:R_0805_2012Metric_Pad1.20x1.40mm_HandSolder
- moved G*** 106.2 mm to (322.9, 146.8)
- moved logo1 90.2 mm to (291.9, 147.2)
- moved R1 0.55 mm to (310.7, 81.9)
Connections:
- SW17 pad S1: Net-(D17-A) -> C16
- SW17 pad S2: C16 -> Net-(D17-A)
Routing:
- net GND: track 357.0 -> 368.6 mm
- net C10: track 206.6 -> 202.7 mm
- net C11: track 228.2 -> 224.6 mm
- net C6: track 125.8 -> 122.3 mm
- net C13: track 281.1 -> 277.6 mm
- net C12: track 248.7 -> 245.2 mm
- net C16: track 337.7 -> 335.7 mm
- net C9: track 173.5 -> 172.1 mm
- net C8: track 142.4 -> 141.0 mm
- net R0: track 392.7 -> 393.4 mm
- net Net-(D91-A): track 10.3 -> 9.76 mm
