File: kicad-pcb/krunchboard-v2-plate/krunchboard-90-plate.kicad_pcb (KiCad board)
At the start: 2 copper layers, 334.8 x 130.2 mm, 4 parts

Commit message: updated case,plate (added 4 extra mounting hole in center), updated pcb to prod v1
Parts:
- added REF**: MountingHole_2.2mm_M2, MountingHole:MountingHole_2.2mm_M2, F.Cu at (202.7, 194.5)
- added REF**: MountingHole_2.2mm_M2, MountingHole:MountingHole_2.2mm_M2, F.Cu at (216.7, 194.6)
- added REF**: MountingHole_2.2mm_M2, MountingHole:MountingHole_2.2mm_M2, F.Cu at (216.7, 65.9)
- added REF**: MountingHole_2.2mm_M2, MountingHole:MountingHole_2.2mm_M2, F.Cu at (202.7, 65.9)
Other:
- board size 334.8 x 130.2 mm -> 334.8 x 136.5 mm
